File: EAGLE files/Projects/AB_BOARD_V1.sch (EAGLE design)
At the start: 23 parts

Commit message: update AB_board_schem_V1
Parts:
- added J2: (no value), Sightline:JST_GH_SM06B-GHS-TB
- added J3: (no value), Sightline:MOLEX_53048-03
- added J4: (no value), Sightline:MOLEX_53398-04
- added R3, R4, R5, R6, R7: 0, SparkFun-Resistors:RESISTOR0402
- added X1: 53048-03, con-molex:53048-03
- C1, C2, C3, C5: value CAP3216-18LOW_ESR -> 10uf
- C10, C11, C12, C13, C14, C15, C16, C17, C6, C7, C8, C9: value (none) -> 100nf
- C4: value CAP3216-18LOW_ESR -> 10u
Connections:
- new net N$17: J1.RXC, J2.2, J3.RX
- new net N$18: J1.TXC, J2.3, J3.TX
- new net N$19: J2.4, R3.2, R5.2, R6.1
- new net N$20: J2.5, R4.2, R5.1, R7.1
- new net N$21: J1.UART_RX_CAM, R6.2
- new net N$22: J1.UART_TX_CAM, R7.2
- new net N$23: J1.CAM_GPIO172, J4.GPIO172
- new net N$24: J1.CAM_GPIO173, J4.GPIO173
- new net N$25: J1.CAM_GPIO175, J4.GPIO175
- net +5V: now also J2.1
- net GND: now also J2.6, J3.GND, J4.GND
- net I2C_SCL: now also R3.1
- net I2C_SDA: now also R4.1
Other:
- note added: "DNP"
