File: EAGLE files/Projects/SLA_1500_CAM_V2.sch (EAGLE design)
At the start: 63 parts, among them J5 MOLEX 53398-04

Commit message: Update SLA_1500_CAM
Changed lines of the file:
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@@
 <setting verticaltext="up"/>
 </settings>
-<grid distance="0.1" unitdist="inch" unit="inch" style="lines" multiple="1" display="yes" altdistance="0.01" altunitdist="inch" altunit="inch"/>
+<grid distance="0.1" unitdist="inch" unit="inch" style="lines" multiple="1" display="no" altdistance="0.01" altunitdist="inch" altunit="inch"/>
 <layers>
 <layer number="1" name="Top" color="4" fill="1" visible="yes" active="no"/>
@@
 </classes>
 <parts>
-<part name="FRAME1" library="frames" library_urn="urn:adsk.eagle:library:229" deviceset="FRAME_B_L" device=""/>
+<part name="FRAME1" library="frames" library_urn="urn:adsk.eagle:library:229" deviceset="FRAME_B_L" device="">
+<attribute name="SPICEPREFIX" value="X"/>
+</part>
 <part name="C7" library="Sightline" deviceset="CAP0201" device="100NF" package3d_urn="urn:adsk.eagle:package:26117/2" value="100nf"/>
 <part name="C8" library="Sightline" deviceset="CAP0201" device="100NF" package3d_urn="urn:adsk.eagle:package:26117/2" value="100nf"/>
@@
 <part name="LED1" library="led" library_urn="urn:adsk.eagle:library:259" deviceset="LED" device="CHIP-LED0603" package3d_urn="urn:adsk.eagle:package:15819/3"/>
 <part name="GND31" library="supply1" library_urn="urn:adsk.eagle:library:371" deviceset="GND" device=""/>
+<part name="U$1" library="Sightline" deviceset="HEADER_V2" device=""/>
 </parts>
 <sheets>
@@
 <instances>
 <instance part="FRAME1" gate="G$1" x="0" y="0.2" smashed="yes"/>
-<instance part="FRAME1" gate="G$2" x="325.12" y="0.2" smashed="yes">
-<attribute name="LAST_DATE_TIME" x="337.82" y="1.47" size="2.54" layer="94"/>
-<attribute name="SHEET" x="411.48" y="1.47" size="2.54" layer="94"/>
-<attribute name="DRAWING_NAME" x="342.9" y="19.25" size="2.54" layer="94"/>
-</instance>
 <instance part="C7" gate="G$1" x="327.66" y="246.38" smashed="yes"/>
 <instance part="C8" gate="G$1" x="317.5" y="246.38" smashed="yes"/>
@@
 </instance>
 <instance part="J1" gate="G$1" x="256.54" y="129.54" smashed="yes">
-<attribute name="NAME" x="254" y="157.48" size="1.778" layer="95" rot="R180" align="top-right"/>
+<attribute name="NAME" x="241.3" y="165.1" size="1.778" layer="95" rot="R180" align="top-right"/>
 </instance>
 <instance part="GND8" gate="1" x="281.94" y="91.44" smashed="yes">
@@
 <attribute name="VALUE" x="358.14" y="223.52" size="1.778" layer="96"/>
 </instance>
+<instance part="U$1" gate="G$1" x="322.58" y="2.54" smashed="yes"/>
 </instances>
 <busses>

Commit message: Update SLA_1500_CAM
Other:
- note added: "AUXILLARY POWER IN"
- note removed: "AUXILLARY POWER"
Changed lines of the file:
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@@
 <grid distance="0.1" unitdist="inch" unit="inch" style="lines" multiple="1" display="no" altdistance="0.01" altunitdist="inch" altunit="inch"/>
 <layers>
-<layer number="1" name="Top" color="4" fill="1" visible="yes" active="no"/>
-<layer number="2" name="Route2" color="1" fill="3" visible="yes" active="no"/>
-<layer number="3" name="Route3" color="4" fill="3" visible="yes" active="no"/>
-<layer number="4" name="Route4" color="1" fill="4" visible="yes" active="no"/>
-<layer number="5" name="Route5" color="4" fill="4" visible="yes" active="no"/>
-<layer number="6" name="Route6" color="1" fill="8" visible="yes" active="no"/>
-<layer number="7" name="Route7" color="4" fill="8" visible="yes" active="no"/>
-<layer number="8" name="Route8" color="1" fill="2" visible="yes" active="no"/>
-<layer number="9" name="Route9" color="4" fill="2" visible="yes" active="no"/>
-<layer number="10" name="Route10" color="1" fill="7" visible="yes" active="no"/>
-<layer number="11" name="Route11" color="4" fill="7" visible="yes" active="no"/>
-<layer number="12" name="Route12" color="1" fill="5" visible="yes" active="no"/>
-<layer number="13" name="Route13" color="4" fill="5" visible="yes" active="no"/>
-<layer number="14" name="Route14" color="1" fill="6" visible="yes" active="no"/>
-<layer number="15" name="Route15" color="4" fill="6" visible="yes" active="no"/>
-<layer number="16" name="Bottom" color="1" fill="1" visible="yes" active="no"/>
-<layer number="17" name="Pads" color="2" fill="1" visible="yes" active="no"/>
-<layer number="18" name="Vias" color="2" fill="1" visible="yes" active="no"/>
-<layer number="19" name="Unrouted" color="6" fill="1" visible="yes" active="no"/>
-<layer number="20" name="Dimension" color="15" fill="1" visible="yes" active="no"/>
-<layer number="21" name="tPlace" color="7" fill="1" visible="yes" active="no"/>
-<layer number="22" name="bPlace" color="7" fill="1" visible="yes" active="no"/>
-<layer number="23" name="tOrigins" color="15" fill="1" visible="yes" active="no"/>
-<layer number="24" name="bOrigins" color="15" fill="1" visible="yes" active="no"/>
-<layer number="25" name="tNames" color="7" fill="1" visible="yes" active="no"/>
-<layer number="26" name="bNames" color="7" fill="1" visible="yes" active="no"/>
-<layer number="27" name="tValues" color="7" fill="1" visible="yes" active="no"/>
-<layer number="28" name="bValues" color="7" fill="1" visible="yes" active="no"/>
+<layer number="1" name="Top" color="4" fill="1" visible="no" active="no"/>
+<layer number="2" name="Route2" color="1" fill="3" visible="no" active="no"/>
+<layer number="3" name="Route3" color="4" fill="3" visible="no" active="no"/>
+<layer number="4" name="Route4" color="1" fill="4" visible="no" active="no"/>
+<layer number="5" name="Route5" color="4" fill="4" visible="no" active="no"/>
+<layer number="6" name="Route6" color="1" fill="8" visible="no" active="no"/>
+<layer number="7" name="Route7" color="4" fill="8" visible="no" active="no"/>
+<layer number="8" name="Route8" color="1" fill="2" visible="no" active="no"/>
+<layer number="9" name="Route9" color="4" fill="2" visible="no" active="no"/>
+<layer number="10" name="Route10" color="1" fill="7" visible="no" active="no"/>
+<layer number="11" name="Route11" color="4" fill="7" visible="no" active="no"/>
+<layer number="12" name="Route12" color="1" fill="5" visible="no" active="no"/>
+<layer number="13" name="Route13" color="4" fill="5" visible="no" active="no"/>
+<layer number="14" name="Route14" color="1" fill="6" visible="no" active="no"/>
+<layer number="15" name="Route15" color="4" fill="6" visible="no" active="no"/>
+<layer number="16" name="Bottom" color="1" fill="1" visible="no" active="no"/>
+<layer number="17" name="Pads" color="2" fill="1" visible="no" active="no"/>
+<layer number="18" name="Vias" color="2" fill="1" visible="no" active="no"/>
+<layer number="19" name="Unrouted" color="6" fill="1" visible="no" active="no"/>
+<layer number="20" name="Dimension" color="15" fill="1" visible="no" active="no"/>
+<layer number="21" name="tPlace" color="7" fill="1" visible="no" active="no"/>
+<layer number="22" name="bPlace" color="7" fill="1" visible="no" active="no"/>
+<layer number="23" name="tOrigins" color="15" fill="1" visible="no" active="no"/>
+<layer number="24" name="bOrigins" color="15" fill="1" visible="no" active="no"/>
+<layer number="25" name="tNames" color="7" fill="1" visible="no" active="no"/>
+<layer number="26" name="bNames" color="7" fill="1" visible="no" active="no"/>
+<layer number="27" name="tValues" color="7" fill="1" visible="no" active="no"/>
+<layer number="28" name="bValues" color="7" fill="1" visible="no" active="no"/>
 <layer number="29" name="tStop" color="7" fill="3" visible="no" active="no"/>
 <layer number="30" name="bStop" color="7" fill="6" visible="no" active="no"/>
@@
 <layer number="35" name="tGlue" color="7" fill="4" visible="no" active="no"/>
 <layer number="36" name="bGlue" color="7" fill="5" visible="no" active="no"/>
-<layer number="37" name="tTest" color="7" fill="1" visible="yes" active="no"/>
-<layer number="38" name="bTest" color="7" fill="1" visible="yes" active="no"/>
+<layer number="37" name="tTest" color="7" fill="1" visible="no" active="no"/>
+<layer number="38" name="bTest" color="7" fill="1" visible="no" active="no"/>
 <layer number="39" name="tKeepout" color="4" fill="11" visible="no" active="no"/>
 <layer number="40" name="bKeepout" color="1" fill="11" visible="no" active="no"/>
@@
 <layer number="44" name="Drills" color="7" fill="1" visible="no" active="no"/>
 <layer number="45" name="Holes" color="7" fill="1" visible="no" active="no"/>
-<layer number="46" name="Milling" color="3" fill="1" visible="yes" active="no"/>
-<layer number="47" name="Measures" color="7" fill="1" visible="yes" active="no"/>
-<layer number="48" name="Document" color="7" fill="1" visible="yes" active="no"/>
-<layer number="49" name="Reference" color="7" fill="1" visible="yes" active="no"/>
-<layer number="50" name="dxf" color="7" fill="1" visible="yes" active="no"/>
-<layer number="51" name="tDocu" color="7" fill="1" visible="yes" active="no"/>
-<layer number="52" name="bDocu" color="7" fill="1" visible="yes" active="no"/>
-<layer number="53" name="tGND_GNDA" color="7" fill="9" visible="yes" active="no"/>
-<layer number="54" name="bGND_GNDA" color="1" fill="9" visible="yes" active="no"/>
-<layer number="56" name="wert" color="7" fill="1" visible="yes" active="no"/>
-<layer number="57" name="tCAD" color="7" fill="1" visible="yes" active="no"/>
-<layer number="59" name="tCarbon" color="7" fill="1" visible="yes" active="no"/>
-<layer number="60" name="bCarbon" color="7" fill="1" visible="yes" active="no"/>
+<layer number="46" name="Milling" color="3" fill="1" visible="no" active="no"/>
+<layer number="47" name="Measures" color="7" fill="1" visible="no" active="no"/>
+<layer number="48" name="Document" color="7" fill="1" visible="no" active="no"/>
+<layer number="49" name="Reference" color="7" fill="1" visible="no" active="no"/>
+<layer number="50" name="dxf" color="7" fill="1" visible="no" active="no"/>
+<layer number="51" name="tDocu" color="7" fill="1" visible="no" active="no"/>
+<layer number="52" name="bDocu" color="7" fill="1" visible="no" active="no"/>
+<layer number="53" name="tGND_GNDA" color="7" fill="9" visible="no" active="no"/>
+<layer number="54" name="bGND_GNDA" color="1" fill="9" visible="no" active="no"/>
+<layer number="56" name="wert" color="7" fill="1" visible="no" active="no"/>
+<layer number="57" name="tCAD" color="7" fill="1" visible="no" active="no"/>
+<layer number="59" name="tCarbon" color="7" fill="1" visible="no" active="no"/>
+<layer number="60" name="bCarbon" color="7" fill="1" visible="no" active="no"/>
 <layer number="88" name="SimResults" color="9" fill="1" visible="yes" active="yes"/>
 <layer number="89" name="SimProbes" color="9" fill="1" visible="yes" active="yes"/>
@@
 <text x="370.84" y="137.16" size="1.778" layer="97" rot="R180" align="center-right">DNP</text>
 <text x="363.22" y="144.78" size="1.778" layer="97" rot="R180" align="center-left">DNP</text>
-<text x="345.44" y="68.58" size="1.778" layer="97">AUXILLARY POWER</text>
+<text x="345.44" y="68.58" size="1.778" layer="97">AUXILLARY POWER IN</text>
 <text x="345.44" y="93.98" size="1.778" layer="97">AUXILLARY I2C BUS TO SIGHTLINE</text>
 <text x="345.44" y="121.92" size="1.778" layer="97">DISCRETE GPIO</text>

Commit message: Update SLA_1500_CAM
Parts:
- removed C15, C16: 100nf, Sightline:CAP0201100NF
- removed R3, R4, R5, R6, R7: 0, SparkFun-Resistors:RESISTOR0402
- added C32, C33: 100nf, Seeed-Capacitor:CERAMIC-100NF-25V-10%-X7R(0402)
- added C34, C35: (no value), Sightline:CAP0201100NF
- added R12, R13, R14: 0, SparkFun-Resistors:RESISTOR0402
- added U8: TXB0104RUTR, Sightline:TXB0104RUTR
- C10, C11, C12, C13, C14, C7, C8, C9: value 100nf -> (none)
Connections:
- new net N$13: C10.P$1, C11.P$1, C12.P$1, C18.+, C3.+, JP3.2
- new net N$31: J1.AGND2, R12.1
- new net N$32: R13.2, U1.TRIGGER
- new net N$33: R14.2, U1.FLASH
- new net N$34: J1.TXC, U8.A2
- new net N$36: J2.4, U8.B3
- new net P3P8V: C33.1, U8.VCC_B
- new net STANDBY: J1.CAM_GPIO178, U1.STANDBY
- net CAM_GPIO172: now also R13.1
- net CAM_GPIO173: now also R14.1
- net GND: now also C32.1, C33.2, C34.P$2, C35.P$2, R12.2, U8.GND; no longer C15.P$2, C16.P$2, J1.AGND2
- net I2C_SCL: now also U8.A3; no longer R3.1
- net I2C_SDA: now also U8.A4; no longer R4.1
- net N$17: now also J1.RXC, U8.A1; no longer J2.4, R3.2, R5.2, R6.2
- net N$18: now also J2.3, J3.2, U8.B2; no longer J2.5, R4.2, R5.1, R7.2
- net N$19: now also J2.5, U8.B4; no longer J1.RXC, J2.2, J3.3
- net N$20: now also J2.2, J3.3, U8.B1; no longer J1.TXC, J2.3, J3.2
- net P1P8V: now also C32.2, U8.OE, U8.VCC_A
- net SLA_RESET_BAR: now also J1.CAM_GPIO174
- net UART_RX_CAM: no longer R6.1
- net UART_TX_CAM: no longer R7.1
- net VAA: no longer C11.P$1, C12.P$1, C13.P$1, C18.+, C3.+, JP3.2
- net VAA_PIX: now also C13.P$1; no longer C15.P$1
- net VDD: now also C34.P$1, C35.P$1; no longer C10.P$1, C9.P$1
- net VDD_PLL: now also C9.P$1; no longer C16.P$1
Other:
- note added: "TO 1500-OEM J4"
- moved on the sheet: C30, C31, J2, J3, J4, J5, J6, R10, S1, U6, U7
