File: EAGLE files/Projects/SLA_1500_CAM_V2.sch (EAGLE design)
At the start: 71 parts, among them J4 MOLEX 53398-0471, J5 MOLEX 53398-04, U8 TXB0104RUTR

Commit message: Update SLA 1500 CAM V2
Connections:
- removed net N$13: C10.P$1, C11.P$1, C12.P$1, C18.+, C3.+, JP3.2
- net VAA: now also C10.P$1, C11.P$1, C12.P$1, C18.+, C3.+, JP3.2
