File: EAGLE files/Projects/SLA_1500_CAM_V4.brd (EAGLE design)
At the start: 37.8 x 26.4 mm, 91 parts, among them J2 JST GH SM06B, J3 MOLEX 53261-03, J4 MOLEX 53261-04, J5 MOLEX 53261-04, J6 MOLEX 53261-04, U11 TXS0102, U2 TPS73633DCQR, U8 TXS0102, U9 TXS0102

Commit message: Update SLA1500 CAM V4
Connections:
- removed net CAM_GPIO175: J4.4
- new net CAM_GPIO178: J1.19, J4.4
Changed lines of the file:
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@@
 <wire x1="9.5292" y1="43.5102" x2="-21.5538" y2="7.5592" width="0" layer="19" extent="1-1"/>
-</signal>
-<signal name="CAM_GPIO175">
-<contactref element="J4" pad="4"/>
 </signal>
 <signal name="P5V">
@@
 <wire x1="13.716" y1="-1.25" x2="13.6798" y2="-4.0232" width="0" layer="19" extent="16-16"/>
 </signal>
+<signal name="CAM_GPIO178">
+<contactref element="J4" pad="4"/>
+<contactref element="J1" pad="19"/>
+<wire x1="1.4746" y1="-6.963" x2="-21.5538" y2="8.8092" width="0" layer="19" extent="1-16"/>
+</signal>
 </signals>
