File: EAGLE files/Projects/SLA_1500_CAM_V4.brd (EAGLE design)
At the start: 37.8 x 26.4 mm, 97 parts, among them J2 JST GH SM06B, J3 MOLEX 53261-03, J4 MOLEX 53261-04, J5 MOLEX 53261-04, J6 MOLEX 53261-04, U10 TPS73633DBVR, U11 TXS0102, U8 TXS0102, U9 TXS0102

Commit message: Update SLA1500 CAM V4 .brd
Parts:
- moved R23 25.4 mm to (-5.56, -18.8), turned to 0 degrees
- moved R21 20.5 mm to (-9.88, -18.5), turned to 0 degrees
- moved R22 5.70 mm to (-24.6, -6.45), turned to 0 degrees
- moved R17 5.54 mm to (-24.5, -8.99), turned to 0 degrees
- moved R24 5.47 mm to (-24.3, -3.76), turned to 0 degrees
- moved R26 4.68 mm to (2.21, -14.0), turned to 0 degrees
- moved R4 4.03 mm to (1.65, -13.3), turned to 0 degrees
- moved R6 3.63 mm to (1.14, -12.6), turned to 0 degrees
- moved R15 2.41 mm to (0.66, -9.25), turned to 0 degrees
Routing:
- net SLA_RESET_BAR: track 0.00 -> 33.9 mm, vias 0 -> 4
- net N$36: track 0.00 -> 16.3 mm, vias 0 -> 2
- net N$45: track 0.00 -> 10.0 mm, vias 0 -> 2
- net N$10: track 0.01 -> 9.25 mm
- net N$3: track 0.04 -> 8.47 mm, vias 0 -> 1
- net N$7: track 0.00 -> 8.42 mm, vias 0 -> 1
- net N$35: track 0.00 -> 6.97 mm
- net N$11: track 0.00 -> 5.36 mm, vias 0 -> 1
- net N$2: track 4.57 -> 9.50 mm
- net N$24: track 0.00 -> 4.88 mm, vias 0 -> 1
- net N$6: track 4.57 -> 9.18 mm
- net P1P8V: track 45.2 -> 48.3 mm
- net N$22: track 4.57 -> 6.70 mm
- net CAM_GPIO172: track 52.0 -> 53.2 mm
- net N$1: track 6.45 -> 7.52 mm
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
Commit message: Update SLA1500 CAM V4 .brd
Parts:
- moved R17 24.8 mm to (0.13, -6.53), turned to 180 degrees
- moved R24 16.9 mm to (-7.62, -1.35), turned to 180 degrees
- moved R23 16.8 mm to (-11.0, -2.90), turned to 180 degrees
- moved R21 14.4 mm to (-11.0, -4.17), turned to 180 degrees
- moved R22 13.9 mm to (-11.0, -3.53)
- moved R19 1.81 mm to (-9.42, -1.73), turned to 180 degrees
- moved C13 1.06 mm to (2.54, -2.57), turned to 180 degrees
- moved R3 0.86 mm to (1.12, -5.21)
- moved R5 0.85 mm to (-0.48, -5.56)
- moved R7 0.84 mm to (-1.32, -6.91)
Routing:
- net N$47: track 0.00 -> 27.6 mm
- net N$43: track 0.00 -> 24.5 mm
- net N$49: track 0.00 -> 21.9 mm, vias 0 -> 2
- net N$40: track 0.00 -> 15.8 mm, vias 0 -> 1
- net N$45: track 10.0 -> 18.9 mm
- net N$46: track 0.00 -> 8.60 mm, vias 0 -> 1
- net N$44: track 0.00 -> 8.58 mm, vias 0 -> 1
- net N$35: track 6.97 -> 14.5 mm
- net N$42: track 0.00 -> 6.71 mm, vias 0 -> 1
- net N$36: track 16.3 -> 19.8 mm
- net N$41: track 0.00 -> 3.02 mm
- net N$48: track 0.00 -> 2.99 mm, vias 0 -> 1
- net N$53: track 10.7 -> 13.5 mm
- net P2P8V: track 22.9 -> 25.4 mm
- net N$8: track 3.62 -> 2.10 mm
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