File: EAGLE files/Projects/SLA_1500_CAM_V5.brd (EAGLE design)
At the start: 37.8 x 26.4 mm, 97 parts, among them J2 JST GH SM06B, J3 MOLEX 53261-03, J4 MOLEX 53261-04, J5 MOLEX 53261-04, J6 MOLEX 53261-04, U10 TPS73633DBVR, U11 TXS0102, U8 TXS0102, U9 TXS0102

Commit message: Update SLA1500 CAM V5 .brd
Parts:
- R16, R20: device SparkFun-Resistors:0603 -> resistor:R0201
- moved R20 21.1 mm to (-6.20, 3.81)
- moved R16 20.7 mm to (-6.68, 2.24), turned to 180 degrees
- moved R26 15.3 mm to (1.24, -9.32)
- moved R4 14.3 mm to (0.20, -9.30)
- moved R6 13.2 mm to (-0.79, -9.30)
- moved R3 12.8 mm to (-2.13, -6.15)
- moved R17 12.7 mm to (-0.71, -5.16), turned to 0 degrees
- moved R5 11.9 mm to (-2.13, -5.54)
- moved R15 11.7 mm to (-1.75, -9.73)
- moved R7 10.1 mm to (-1.45, -7.62)
- moved C15 9.35 mm to (4.60, 5.94)
- moved R2 9.12 mm to (0.43, 3.63)
- moved U5 9.02 mm to (1.98, 6.68)
- moved R1 7.04 mm to (5.44, 8.86)
- moved C44 4.76 mm to (-9.35, 2.41)
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Connections:
- net I2C_SCL: now also R20.1; no longer R16.1
- net I2C_SDA: now also R16.1; no longer R20.1
Routing:
- net I2C_SDA: track 1.33 -> 30.6 mm, vias 1 -> 3
- net N$47: track 1.33 -> 28.1 mm, vias 1 -> 2
- net I2C_SCL: track 0.15 -> 24.9 mm, vias 0 -> 2
- net CAM_GPIO173: track 8.53 -> 32.0 mm, vias 2 -> 4
- net SLA_RESET_BAR: track 5.36 -> 27.6 mm, vias 2 -> 4
- net CAM_GPIO178: track 0.77 -> 22.2 mm, vias 0 -> 3
- net N$36: track 0.00 -> 19.9 mm, vias 0 -> 4
- net N$43: track 0.00 -> 19.2 mm, vias 0 -> 2
- net N$49: track 0.27 -> 18.7 mm, vias 0 -> 2
- net N$53: track 0.01 -> 16.4 mm
- net N$35: track 0.04 -> 14.7 mm
- net N$40: track 0.00 -> 12.3 mm, vias 0 -> 1
- net N$3: track 1.33 -> 10.7 mm
- net P2P8V: track 23.1 -> 16.2 mm, vias 8 -> 7
- net N$1: track 0.00 -> 6.41 mm, vias 0 -> 1
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
Commit message: Update SLA1500 CAM V5 .brd
Parts:
- moved R12 6.28 mm to (-9.55, -14.1), flipped to the top
- moved C14 4.01 mm to (-0.99, 0.23)
- moved R5 1.80 mm to (-0.86, -4.27)
- moved R3 1.71 mm to (-0.91, -4.95)
- moved R17 1.58 mm to (-0.89, -3.58)
- moved R23 1.21 mm to (-11.3, -1.73)
- moved R22 1.02 mm to (-11.0, -2.51), turned to 180 degrees
- moved R21 0.99 mm to (-11.0, -3.17)
- moved R26 0.86 mm to (1.96, -9.80)
- moved R4 0.82 mm to (0.86, -9.78)
- moved R7 0.77 mm to (-1.68, -6.88)
- moved R6 0.53 mm to (-0.56, -9.78)
Routing:
- net CAM_GPIO172: track 3.40 -> 44.9 mm, vias 0 -> 3
- net N$45: track 0.00 -> 19.1 mm, vias 0 -> 2
- net P5V: track 26.9 -> 18.9 mm, vias 8 -> 7
- net FRAME_VALID: track 25.8 -> 33.6 mm
- net N$46: track 0.00 -> 7.17 mm, vias 0 -> 1
- net N$44: track 0.05 -> 6.46 mm, vias 0 -> 1
- net N$42: track 0.00 -> 6.30 mm, vias 0 -> 1
- net N$35: track 14.7 -> 20.7 mm
- net N$31: track 0.07 -> 6.07 mm
- net I2C_SCL: track 24.9 -> 30.8 mm
- net LINE_VALID: track 20.4 -> 26.1 mm
- net I2C_SDA: track 30.6 -> 36.0 mm
- net SLA_RESET_BAR: track 27.6 -> 32.4 mm
- net STANDBY: track 16.9 -> 21.7 mm
- net N$49: track 18.7 -> 23.0 mm
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
Commit message: Update SLA1500 CAM V5 .brd
Parts:
- removed C28, C29: 10uf, Seeed-Capacitor:AVX-A
- removed TP4, TP5, TP6, TP7, TP8: PTR1PAD1-13, testpad:P1-13
- added C17, C6: 10uf, Sightline:0402
- C1, C18, C19, C2, C20, C3, C4, C5: device Seeed-Capacitor:AVX-A -> Sightline:0402
- TP1, TP2, TP3: value PTR1PAD1-13 -> PTR1TP08SQ; device testpad:P1-13 -> testpad:TP08SQ
- moved TP3 32.3 mm to (8.46, -14.1)
- moved TP2 29.1 mm to (10.5, -14.1)
- moved C20 28.5 mm to (-4.78, 3.40)
- moved TP1 23.0 mm to (-17.9, -4.45)
- moved C2 16.5 mm to (9.55, -4.09), flipped to the bottom, turned to 180 degrees
- moved C18 15.9 mm to (11.9, 10.1), flipped to the bottom
- moved C3 13.5 mm to (11.3, -3.02), flipped to the bottom, turned to 180 degrees
- moved C4 10.00 mm to (13.7, -1.93), flipped to the bottom, turned to 180 degrees
- moved C5 4.96 mm to (12.0, 7.65), turned to 0 degrees
- moved C19 3.23 mm to (-0.69, 9.93), flipped to the top, turned to 180 degrees
- moved C1 2.17 mm to (-9.73, 9.37), flipped to the top, turned to 90 degrees
- moved C30 1.48 mm to (-15.3, 10.3)
- moved C23 0.87 mm to (-15.9, -5.03), turned to 270 degrees
- moved R19 0.68 mm to (-6.73, 0.71)
- moved R23 0.36 mm to (-11.6, -1.88)
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Connections:
- removed net N$53: J1.39, R19.2
- new net CAM_PCLK: J1.39, R19.2, TP1.TP
- net GND: now also C1.2, C17.2, C18.2, C19.2, C2.2, C20.2, C3.2, C4.2, C5.2, C6.2; no longer C1.-, C18.-, C19.-, C2.-, C20.-, C28.-, C29.-, C3.-, C4.-, C5.-, TP8.TP
- net P1P8V: now also C1.1, C19.1, C20.1, C6.1; no longer C1.+, C19.+, C28.+, C5.+, TP7.TP
- net P2P8V: now also C17.1, C18.1, C2.1, C3.1, C4.1, C5.1; no longer C18.+, C2.+, C20.+, C29.+, C3.+, C4.+, TP6.TP
- net P3P3V: no longer TP5.TP
- net P5V: no longer TP4.TP
- net PIXCLK: no longer TP1.TP
Routing:
- net CAM_PCLK: track 0.00 -> 28.3 mm, vias 0 -> 4
- net N$53: track 16.9 -> 0.00 mm
- net P2P8V: track 19.6 -> 29.8 mm, vias 7 -> 12
- net LINE_VALID: track 26.1 -> 34.1 mm, vias 1 -> 2
- net N$28: track 0.00 -> 5.27 mm, vias 0 -> 1
- net P1P8V: track 35.5 -> 40.7 mm, vias 13 -> 14
- net FRAME_VALID: track 33.6 -> 30.6 mm
- net I2C_SCL: track 30.8 -> 27.8 mm
- net PIXCLK: track 0.11 -> 3.06 mm, vias 0 -> 1
- net STANDBY: track 21.7 -> 18.8 mm
- net SLA_RESET_BAR: track 32.4 -> 29.8 mm
- net N$45: track 19.1 -> 20.9 mm
- net CAM_GPIO173: track 31.4 -> 33.1 mm
- net I2C_SDA: track 36.0 -> 34.4 mm
- net P5V: track 18.9 -> 20.3 mm
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