File: EAGLE files/Projects/SLA_1500_CAM_V5.sch (EAGLE design)
At the start: 97 parts, among them J2 JST GH SM06B, J3 MOLEX 53261-03, J4 MOLEX 53261-04, J5 MOLEX 53261-04, J6 MOLEX 53261-04, U10 TPS73633DBVR, U11 TXS0102, U8 TXS0102, U9 TXS0102

Commit message: Update SLA1500 CAM V5 .brd
Parts:
- removed C28, C29: 10uf, Seeed-Capacitor:TANTALUM-SMD-10UF-10V-10%(AVX-A)
- removed TP4, TP5, TP6, TP7, TP8: PTR1PAD1-13, testpad:PTR1PAD1-13
- added C17, C6: 10uf, Sightline:F980G106MUA
- C1, C18, C19, C2, C20, C3, C4, C5: device Seeed-Capacitor:TANTALUM-SMD-10UF-10V-10%(AVX-A) -> Sightline:F980G106MUA
- TP1, TP2, TP3: value PTR1PAD1-13 -> PTR1TP08SQ; device testpad:PTR1PAD1-13 -> testpad:PTR1TP08SQ
Connections:
- removed net N$53: J1.CAM_PCLK, R19.2
- new net CAM_PCLK: J1.CAM_PCLK, R19.2, TP1.TP
- net GND: now also C1.P$2, C17.P$2, C18.P$2, C19.P$2, C2.P$2, C20.P$2, C3.P$2, C4.P$2, C5.P$2, C6.P$2; no longer C1.-, C18.-, C19.-, C2.-, C20.-, C28.-, C29.-, C3.-, C4.-, C5.-, TP8.TP
- net P1P8V: now also C1.P$1, C19.P$1, C20.P$1, C6.P$1; no longer C1.+, C19.+, C28.+, C5.+, TP7.TP
- net P2P8V: now also C17.P$1, C18.P$1, C2.P$1, C3.P$1, C4.P$1, C5.P$1; no longer C18.+, C2.+, C20.+, C29.+, C3.+, C4.+, TP6.TP
- net P3P3V: no longer TP5.TP
- net P5V: no longer TP4.TP
- net PIXCLK: no longer TP1.TP
Other:
- moved on the sheet: TP1, TP2, TP3

Commit message: Update SLA1500 CAM V5 .brd
Other:
- note added: "AUXILIARY POWER IN 5VDC"
- note removed: "AUXILIARY POWER IN"
Changed lines of the file:
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@@
 <part name="D2" library="diode" library_urn="urn:adsk.eagle:library:210" deviceset="BAT60J" device="" package3d_urn="urn:adsk.eagle:package:43461/1"/>
 <part name="D1" library="diode" library_urn="urn:adsk.eagle:library:210" deviceset="BAT60J" device="" package3d_urn="urn:adsk.eagle:package:43461/1"/>
-<part name="U$1" library="Sightline" deviceset="HEADER_V4" device=""/>
 <part name="C36" library="Sightline" deviceset="CAP0201" device="100NF" package3d_urn="urn:adsk.eagle:package:26117/2"/>
 <part name="C37" library="Sightline" deviceset="CAP0201" device="100NF" package3d_urn="urn:adsk.eagle:package:26117/2"/>
@@
 <part name="TP2" library="testpad" library_urn="urn:adsk.eagle:library:385" deviceset="PTR1" device="TP08SQ" package3d_urn="urn:adsk.eagle:package:27960/1"/>
 <part name="TP3" library="testpad" library_urn="urn:adsk.eagle:library:385" deviceset="PTR1" device="TP08SQ" package3d_urn="urn:adsk.eagle:package:27960/1"/>
+<part name="U$1" library="Sightline" deviceset="HEADER_V5" device=""/>
 </parts>
 <sheets>
 <sheet>
 <plain>
-<text x="393.7" y="177.8" size="1.778" layer="97">AUXILIARY POWER IN</text>
+<text x="393.7" y="175.26" size="1.778" layer="97">AUXILIARY POWER IN
+5VDC</text>
 <text x="393.7" y="106.68" size="1.778" layer="97">AUXILIARY I2C BUS
 TO SIGHTLINE</text>
@@
 <attribute name="VALUE" x="366.649" y="152.654" size="1.778" layer="96" rot="R90"/>
 </instance>
-<instance part="U$1" gate="G$1" x="322.58" y="5.08" smashed="yes"/>
 <instance part="C36" gate="G$1" x="309.88" y="193.04" smashed="yes">
 <attribute name="NAME" x="313.69" y="189.23" size="1.27" layer="95"/>
@@
 </instance>
 <instance part="R26" gate="G$1" x="215.9" y="160.02" smashed="yes">
-<attribute name="NAME" x="212.09" y="161.5186" size="1.778" layer="95"/>
-<attribute name="VALUE" x="212.09" y="156.718" size="1.778" layer="96"/>
+<attribute name="NAME" x="207.01" y="158.9786" size="1.778" layer="95"/>
+<attribute name="VALUE" x="219.71" y="159.258" size="1.778" layer="96"/>
 </instance>
 <instance part="R3" gate="G$1" x="215.9" y="157.48" smashed="yes">
-<attribute name="NAME" x="212.09" y="158.9786" size="1.778" layer="95"/>
-<attribute name="VALUE" x="212.09" y="154.178" size="1.778" layer="96"/>
+<attribute name="NAME" x="207.01" y="156.4386" size="1.778" layer="95"/>
+<attribute name="VALUE" x="219.71" y="156.718" size="1.778" layer="96"/>
 </instance>
 <instance part="R4" gate="G$1" x="215.9" y="154.94" smashed="yes">
-<attribute name="NAME" x="212.09" y="156.4386" size="1.778" layer="95"/>
-<attribute name="VALUE" x="212.09" y="151.638" size="1.778" layer="96"/>
+<attribute name="NAME" x="207.01" y="153.8986" size="1.778" layer="95"/>
+<attribute name="VALUE" x="219.71" y="154.178" size="1.778" layer="96"/>
 </instance>
 <instance part="R5" gate="G$1" x="215.9" y="152.4" smashed="yes">
-<attribute name="NAME" x="212.09" y="153.8986" size="1.778" layer="95"/>
-<attribute name="VALUE" x="212.09" y="149.098" size="1.778" layer="96"/>
+<attribute name="NAME" x="207.01" y="151.3586" size="1.778" layer="95"/>
+<attribute name="VALUE" x="219.71" y="151.638" size="1.778" layer="96"/>
 </instance>
 <instance part="R6" gate="G$1" x="215.9" y="149.86" smashed="yes">
-<attribute name="NAME" x="212.09" y="151.3586" size="1.778" layer="95"/>
-<attribute name="VALUE" x="212.09" y="146.558" size="1.778" layer="96"/>
+<attribute name="NAME" x="207.01" y="148.8186" size="1.778" layer="95"/>
+<attribute name="VALUE" x="219.71" y="149.098" size="1.778" layer="96"/>
 </instance>
 <instance part="R7" gate="G$1" x="215.9" y="147.32" smashed="yes">
-<attribute name="NAME" x="212.09" y="148.8186" size="1.778" layer="95"/>
-<attribute name="VALUE" x="212.09" y="144.018" size="1.778" layer="96"/>
+<attribute name="NAME" x="207.01" y="146.2786" size="1.778" layer="95"/>
+<attribute name="VALUE" x="219.71" y="146.558" size="1.778" layer="96"/>
 </instance>
 <instance part="R15" gate="G$1" x="215.9" y="144.78" smashed="yes">
-<attribute name="NAME" x="212.09" y="146.2786" size="1.778" layer="95"/>
-<attribute name="VALUE" x="212.09" y="141.478" size="1.778" layer="96"/>
+<attribute name="NAME" x="207.01" y="143.7386" size="1.778" layer="95"/>
+<attribute name="VALUE" x="219.71" y="144.018" size="1.778" layer="96"/>
 </instance>
 <instance part="R17" gate="G$1" x="215.9" y="142.24" smashed="yes">
-<attribute name="NAME" x="212.09" y="143.7386" size="1.778" layer="95"/>
-<attribute name="VALUE" x="212.09" y="138.938" size="1.778" layer="96"/>
+<attribute name="NAME" x="207.01" y="141.1986" size="1.778" layer="95"/>
+<attribute name="VALUE" x="219.71" y="141.478" size="1.778" layer="96"/>
 </instance>
 <instance part="R21" gate="G$1" x="215.9" y="139.7" smashed="yes">
-<attribute name="NAME" x="212.09" y="141.1986" size="1.778" layer="95"/>
-<attribute name="VALUE" x="212.09" y="136.398" size="1.778" layer="96"/>
+<attribute name="NAME" x="207.01" y="138.6586" size="1.778" layer="95"/>
+<attribute name="VALUE" x="219.71" y="138.938" size="1.778" layer="96"/>
 </instance>
 <instance part="R22" gate="G$1" x="215.9" y="137.16" smashed="yes">
-<attribute name="NAME" x="212.09" y="138.6586" size="1.778" layer="95"/>
-<attribute name="VALUE" x="212.09" y="133.858" size="1.778" layer="96"/>
+<attribute name="NAME" x="207.01" y="136.1186" size="1.778" layer="95"/>
+<attribute name="VALUE" x="219.71" y="136.398" size="1.778" layer="96"/>
 </instance>
 <instance part="R23" gate="G$1" x="215.9" y="134.62" smashed="yes">
-<attribute name="NAME" x="212.09" y="136.1186" size="1.778" layer="95"/>
-<attribute name="VALUE" x="212.09" y="131.318" size="1.778" layer="96"/>
+<attribute name="NAME" x="207.01" y="133.5786" size="1.778" layer="95"/>
+<attribute name="VALUE" x="219.71" y="133.858" size="1.778" layer="96"/>
 </instance>
 <instance part="R24" gate="G$1" x="215.9" y="132.08" smashed="yes">
-<attribute name="NAME" x="212.09" y="133.5786" size="1.778" layer="95"/>
-<attribute name="VALUE" x="212.09" y="128.778" size="1.778" layer="96"/>
+<attribute name="NAME" x="207.01" y="131.0386" size="1.778" layer="95"/>
+<attribute name="VALUE" x="219.71" y="131.318" size="1.778" layer="96"/>
 </instance>
 <instance part="U10" gate="G$1" x="58.42" y="208.28" smashed="yes">
@@
 <attribute name="TP_SIGNAL_NAME" x="217.17" y="45.72" size="1.778" layer="97" rot="R180"/>
 </instance>
+<instance part="U$1" gate="G$1" x="322.58" y="5.08" smashed="yes"/>
 </instances>
 <busses>
