File: EAGLE files/Projects/SLA_1500_CAM_V6.brd (EAGLE design)
At the start: 37.8 x 26.4 mm, 92 parts, among them J2 JST GH SM06B, J3 MOLEX 53261-03, J4 MOLEX 53261-04, J5 MOLEX 53261-04, J6 MOLEX 53261-04, U10 TPS73633DBVR, U11 TXS0102, U8 TXS0102, U9 TXS0102

Commit message: Update SLA1500 CAM V6
Parts:
- added C28: 100nF, Seeed-Capacitor:C0402
- added C29: 10nf, Seeed-Capacitor:C0402
- added R25: 0R, Seeed-Resistor:R0402
- added R27: 1.5K, Seeed-Resistor:R0402
- added R28: 22R, Seeed-Resistor:R0402
- added R29: (no value), resistor:R0402
- moved C42 36.3 mm to (27.7, -15.0)
- moved C41 36.3 mm to (27.2, -12.4)
- moved U9 36.3 mm to (27.9, -13.8)
- moved J2 34.9 mm to (23.3, -23.1)
- moved R17 15.6 mm to (7.29, -16.9)
- moved R5 14.4 mm to (6.02, -16.9)
- moved R3 13.3 mm to (4.85, -16.9)
- moved R7 11.4 mm to (3.48, -17.0)
- moved J1 10.4 mm to (0.58, -21.3), turned to 90 degrees
- moved D1 9.92 mm to (-14.5, -19.0)
- moved R6 8.74 mm to (-1.30, -18.5)
- moved R26 8.66 mm to (1.83, -18.5)
- moved R4 7.70 mm to (1.78, -17.4)
- moved R15 7.58 mm to (-1.35, -17.3)
- moved TP2 5.49 mm to (13.5, -18.6)
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Routing:
- net CAM_GPIO172: track 43.7 -> 7.21 mm, vias 3 -> 0
- net N$47: track 29.1 -> 0.00 mm, vias 2 -> 0
- net I2C_SDA: track 34.4 -> 7.30 mm, vias 3 -> 1
- net N$36: track 23.2 -> 0.00 mm, vias 4 -> 0
- net N$49: track 22.6 -> 0.00 mm, vias 2 -> 0
- net N$45: track 20.9 -> 0.08 mm, vias 2 -> 0
- net I2C_SCL: track 27.8 -> 7.16 mm, vias 2 -> 1
- net N$43: track 20.4 -> 0.00 mm, vias 2 -> 0
- net N$35: track 19.4 -> 0.04 mm
- net CAM_PCLK: track 28.3 -> 10.1 mm, vias 4 -> 2
- net LINE_VALID: track 34.1 -> 16.8 mm, vias 2 -> 0
- net SLA_RESET_BAR: track 29.8 -> 16.3 mm, vias 4 -> 3
- net N$40: track 13.4 -> 0.00 mm, vias 1 -> 0
- net STANDBY: track 18.8 -> 5.50 mm, vias 1 -> 0
- net CAM_GPIO173: track 33.1 -> 20.2 mm, vias 4 -> 3
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