File: EAGLE files/Projects/SLA_1500_CAM_V6.brd (EAGLE design)
At the start: 37.8 x 26.4 mm, 98 parts, among them J2 JST GH SM06B, J3 MOLEX 53261-03, J4 MOLEX 53261-04, J5 MOLEX 53261-04, J6 MOLEX 53261-04, U10 TPS73633DBVR, U11 TXS0102, U8 TXS0102, U9 TXS0102

Commit message: Update SLA1500 CAM V6
Parts:
- removed C29: 10nf, Seeed-Capacitor:C0402
- removed C30, C31: 100nf, Seeed-Capacitor:C0402
- removed C42, C43, C44: (no value), Sightline:R0201
- removed R18: 0, SparkFun-Resistors:0402
- removed R20: 1.5k, resistor:R0201
- removed R22, R23, R24, R26: 33R, resistor:R0201
- removed R29: (no value), resistor:R0402
- added C32, C33, C39, C40: 100nF, Seeed-Capacitor:C0402
- added R30, R31, R32: 22R, Seeed-Resistor:R0402
- C10, C11, C12, C13, C14, C15, C16, C34, C35, C36, C37, C41, C7, C8, C9: value (none) -> 100nF; device Sightline:R0201 -> Seeed-Capacitor:C0402
- C27: value 100nf -> 100nF
- R1, R19, R2: value 33 -> 22R; device SparkFun-Resistors:0402 -> Seeed-Resistor:R0402
- R12, R13, R14: value 0 -> 0R; device SparkFun-Resistors:0402 -> Seeed-Resistor:R0402
- R15, R17, R21, R3, R4, R5, R6, R7: value 33R -> 22R; device resistor:R0201 -> Seeed-Resistor:R0402
- R16: value 1.5k -> 1.5K; device resistor:R0201 -> Seeed-Resistor:R0402
- moved R25 40.0 mm to (10.3, -20.0), turned to 180 degrees
- moved C35 35.4 mm to (27.9, -15.3), turned to 270 degrees
- moved C28 33.1 mm to (9.86, -7.11)
- moved R28 32.2 mm to (-7.59, -3.00), turned to 270 degrees
- moved R27 31.4 mm to (-6.99, 1.68), turned to 270 degrees
- moved R12 26.7 mm to (-2.79, 7.26), turned to 270 degrees
- moved C41 26.4 mm to (8.41, 6.07), turned to 90 degrees
- moved C16 23.8 mm to (-15.3, 10.4), flipped to the bottom, turned to 270 degrees
- moved C37 21.3 mm to (-9.12, 2.21), turned to 270 degrees
- moved R19 19.4 mm to (-6.17, -18.6), flipped to the bottom, turned to 0 degrees
- moved R1 18.9 mm to (-9.75, -2.39), turned to 270 degrees
- moved C34 17.9 mm to (9.83, -10.1), turned to 90 degrees
- moved C36 17.6 mm to (27.9, -12.3), turned to 270 degrees
- moved C15 16.4 mm to (-11.8, 5.26), turned to 90 degrees
- moved R2 9.67 mm to (-7.59, -1.75), turned to 270 degrees
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Connections:
- net CAM_GPIO172: now also R13.2; no longer R13.1
- net CAM_GPIO173: now also R14.2; no longer R14.1
- net CAM_PCLK: now also R30.2; no longer R19.2
- net GND: now also C10.1, C11.1, C12.1, C13.1, C14.1, C15.1, C16.1, C28.1, C32.1, C33.1, C34.1, C35.1, C36.1, C37.1, C39.1, C40.1, C41.1, C7.1, C8.1, C9.1, R25.1; no longer C10.2, C11.2, C12.2, C13.2, C14.2, C15.2, C16.2, C30.1, C31.1, C34.2, C35.2, C36.2, C37.2, C41.2, C42.2, C43.2, C44.2, C7.2, C8.2, C9.2, R12.1
- net I2C_SCL: now also R16.1; no longer R20.1
- net I2C_SDA: now also R27.1; no longer R16.1
- net N$10: now also R15.1; no longer R6.1
- net N$11: now also R15.2; no longer R6.2
- net N$12: now also R5.1; no longer R7.1
- net N$14: now also R5.2; no longer R7.2
- net N$15: now also R31.2; no longer R1.2
- net N$16: now also R31.1; no longer R1.1
- net N$2: now also R4.1; no longer R26.1
- net N$22: now also R19.1; no longer R15.1
- net N$24: now also R19.2; no longer R15.2
- net N$25: now also R32.1; no longer R2.1
- net N$26: now also R32.2; no longer R2.2
- net N$3: now also R4.2; no longer R26.2
- net N$31: now also R25.2; no longer R12.2
- net N$32: now also R13.1; no longer R13.2
- net N$33: now also R14.1; no longer R14.2
- net N$4: now also R17.1; no longer R3.1
- net N$40: now also R3.1; no longer R17.1
- net N$41: now also R3.2; no longer R17.2
- net N$42: now also R28.1; no longer R21.1
- net N$43: now also R28.2; no longer R21.2
- net N$44: now also R1.1; no longer R22.1
- net N$45: now also R1.2; no longer R22.2
- net N$46: now also R2.1; no longer R23.1
- net N$47: now also R2.2; no longer R23.2
- net N$48: now also R21.1; no longer R24.1
- net N$49: now also R21.2; no longer R24.2
- net N$5: now also R17.2; no longer R3.2
- net N$52: now also R12.1; no longer R18.1
- net N$6: now also R6.1; no longer R4.1
- net N$7: now also R6.2; no longer R4.2
- net N$8: now also R7.1; no longer R5.1
- net N$9: now also R7.2; no longer R5.2
- net P1P8V: now also C14.2, C27.2, C33.2, C34.2, C36.2, C39.2, C40.2, C7.2, C8.2, R12.2, R27.2; no longer C15.1, C31.2, C34.1, C35.1, C36.1, C41.1, C43.1, C7.1, C8.1, R18.2, R20.2
- net P2P8V: now also C10.2, C11.2, C12.2, C13.2, C32.2, C9.2; no longer C10.1, C11.1, C12.1, C13.1, C14.1, C9.1
- net P3P3V: now also C15.2, C16.2, C28.2, C35.2, C37.2, C41.2; no longer C16.1, C27.2, C30.2, C37.1, C42.1, C44.1
- net PIXCLK: now also R30.1; no longer R19.1
Routing:
- net P3P3V: track 20.8 -> 17.1 mm, vias 6 -> 4
- net N$48: track 2.13 -> 0.00 mm, vias 1 -> 0
- net N$29: track 6.73 -> 5.66 mm
- net I2C_SDA: track 7.30 -> 8.05 mm
- net I2C_SCL: track 7.16 -> 6.49 mm
- net CAM_GPIO173: track 20.2 -> 20.8 mm
- net P1P8V: track 33.4 -> 33.5 mm, vias 11 -> 8
- net GND: vias 7 -> 5

Commit message: Update SLA1500 CAM V6
Parts:
- moved C28 42.3 mm to (-32.1, -12.1)
- moved C34 42.3 mm to (-32.2, -15.1)
- moved J3 42.3 mm to (-25.8, -12.2)
- moved U8 42.3 mm to (-32.1, -13.6)
- moved R21 8.71 mm to (-2.77, -1.17)
- moved R1 6.99 mm to (-2.77, -2.39), turned to 90 degrees
- moved C16 1.49 mm to (-14.1, 9.37)
- moved R2 1.14 mm to (-6.45, -1.78)
- moved R28 0.97 mm to (-6.63, -3.00)
Routing:
- net N$29: track 5.66 -> 6.73 mm
- net P5V: track 15.6 -> 15.1 mm

Commit message: Update SLA1500 CAM V6
Parts:
- removed C17, C19, C4, C6: 10uf, Sightline:0402
- removed C38: 10uf, Seeed-Capacitor:AVX-A
- moved D1 27.9 mm to (12.1, -10.5), turned to 90 degrees
- moved C2 27.8 mm to (-17.3, 3.02), turned to 0 degrees
- moved C28 26.6 mm to (-5.64, -9.46), flipped to the bottom
- moved U8 24.9 mm to (-7.54, -9.84), flipped to the bottom, turned to 0 degrees
- moved C34 24.7 mm to (-8.38, -8.43)
- moved C35 18.8 mm to (10.5, -8.24), flipped to the bottom
- moved C36 18.8 mm to (10.5, -5.27), flipped to the bottom
- moved U9 18.8 mm to (10.5, -6.76), flipped to the bottom
- moved J2 18.7 mm to (15.6, -5.99), flipped to the top, turned to 90 degrees
- moved R3 17.7 mm to (-7.12, -3.86), turned to 270 degrees
- moved R6 15.5 mm to (1.12, -3.51), flipped to the top, turned to 90 degrees
- moved R15 15.4 mm to (-0.66, -3.53), flipped to the top, turned to 90 degrees
- moved J3 15.3 mm to (-10.5, -12.4), flipped to the bottom, turned to 180 degrees
- moved R19 15.0 mm to (-1.30, -4.50), flipped to the top, turned to 90 degrees
- moved R4 14.4 mm to (3.15, -4.50), flipped to the top, turned to 90 degrees
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Connections:
- net GND: no longer C17.2, C19.2, C38.-, C4.2, C6.2
- net P1P8V: no longer C19.1, C6.1
- net P2P8V: no longer C17.1, C2.1, C4.1
- net P5V: now also C2.1; no longer C38.+
Routing:
- net N$41: track 0.00 -> 27.2 mm, vias 0 -> 2
- net N$45: track 0.00 -> 26.6 mm, vias 0 -> 2
- net N$49: track 0.00 -> 25.1 mm
- net LINE_VALID: track 16.8 -> 40.5 mm, vias 0 -> 3
- net FRAME_VALID: track 20.3 -> 43.2 mm, vias 0 -> 3
- net N$36: track 0.00 -> 21.5 mm, vias 0 -> 1
- net CAM_GPIO173: track 20.8 -> 41.0 mm, vias 3 -> 6
- net I2C_SCL: track 6.49 -> 26.1 mm, vias 1 -> 2
- net N$35: track 0.04 -> 18.3 mm, vias 0 -> 1
- net CAM_GPIO178: track 13.2 -> 30.3 mm, vias 2 -> 5
- net CAM_GPIO172: track 7.28 -> 24.3 mm, vias 0 -> 1
- net GND: track 1.69 -> 18.5 mm, vias 5 -> 7
- net I2C_SDA: track 8.05 -> 22.4 mm, vias 1 -> 3
- net STANDBY: track 5.50 -> 18.2 mm, vias 0 -> 3
- net SLA_RESET_BAR: track 16.3 -> 28.0 mm, vias 3 -> 6
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
Commit message: Update SLA1500 CAM V6
Parts:
- moved TP1 31.1 mm to (7.45, -14.2)
- moved TP2 5.20 mm to (10.9, -14.2)
- moved TP3 4.45 mm to (9.08, -14.2)
- moved C37 0.53 mm to (-9.12, 1.68)
- moved U11 0.37 mm to (-9.09, 3.31)
- moved C39 0.34 mm to (-9.14, 4.81)
- moved C34 0.33 mm to (-8.71, -8.43)
- moved C33 0.31 mm to (-2.16, 0.03)
- moved R30 0.28 mm to (-2.12, -0.89)
- moved C7 0.18 mm to (-4.32, 5.77)
- moved C28 0.13 mm to (-5.60, -9.33)
Routing:
- net LINE_VALID: track 40.5 -> 48.2 mm
- net CAM_PCLK: track 16.4 -> 22.4 mm
- net FRAME_VALID: track 43.2 -> 48.1 mm, vias 3 -> 4
- net P3P3V: track 19.4 -> 20.7 mm
- net P1P8V: track 39.8 -> 41.0 mm, vias 12 -> 13
- net GND: vias 7 -> 8

Commit message: Update SLA1500 CAM V6
Parts:
- removed C34, C36, C37, C40: 100nF, Seeed-Capacitor:C0402
- removed R27: 1.5K, Seeed-Resistor:R0402
- removed R28, R30, R31, R32: 22R, Seeed-Resistor:R0402
- added C17: 470nF, SparkFun-Capacitors:0402
- added C19, C30: 100nF, Seeed-Capacitor:C0402
- added C4: 10uf, Sightline:0402
- added R18, R20: 22R, Seeed-Resistor:R0402
- added R22: 60.2K, SparkFun-Resistors:0603
- added R23: 10k, SparkFun-Resistors:0603
- added R24: 0R, Seeed-Resistor:R0402
- C1, C3, C5: value 10uf -> 100nF; device Sightline:0402 -> Seeed-Capacitor:C0402
- C11, C15, C33: value 100nF -> 10uf; device Seeed-Capacitor:C0402 -> Sightline:0402
- C2, C20: value 10uf -> 1uf; device Sightline:0402 -> Seeed-Capacitor:C0402
- C21: value 470nF -> 100nF; device SparkFun-Capacitors:0402 -> Seeed-Capacitor:C0402
- C22: value 10nf -> 100nF
- C23: value 1uf -> 10uf; device Seeed-Capacitor:C0402 -> Sightline:0402
- C25, C26: value 1uf -> 100nF
- C8: value 100nF -> 10nf
- C9: value 100nF -> 1uf
- R1: value 22R -> 10k; device Seeed-Resistor:R0402 -> SparkFun-Resistors:0603
- R10, R9: value 10k -> 22R; device SparkFun-Resistors:0603 -> Seeed-Resistor:R0402
- R11: value 680 -> 22R; device SparkFun-Resistors:0603 -> Seeed-Resistor:R0402
- R12, R13, R14: value 0R -> 22R
- R16: value 1.5K -> 22R
- R25: value 0R -> 680; device Seeed-Resistor:R0402 -> SparkFun-Resistors:0603
- R3, R4: value 22R -> 1.5K
- R6, R7: value 22R -> 0R
- R8: value 60.2K -> 0R; device SparkFun-Resistors:0603 -> Seeed-Resistor:R0402
- moved C24 30.4 mm to (13.2, 5.49)
- moved R25 25.0 mm to (-16.7, 5.05), flipped to the bottom, turned to 180 degrees
- moved D1 24.4 mm to (-11.8, -5.79), flipped to the bottom
- moved D2 24.4 mm to (12.1, -10.5), flipped to the top
- moved C22 22.3 mm to (4.75, -0.01), turned to 270 degrees
- moved C9 21.2 mm to (-15.3, -5.05), turned to 90 degrees
- moved C23 20.6 mm to (2.36, 1.80), turned to 180 degrees
- moved R11 19.8 mm to (1.12, -3.51), flipped to the top, turned to 90 degrees
- moved R2 19.5 mm to (5.21, 8.81), turned to 270 degrees
- moved R10 19.4 mm to (2.11, -9.51), flipped to the bottom, turned to 270 degrees
- moved C21 18.9 mm to (4.77, 0.90), turned to 270 degrees
- moved C20 18.2 mm to (13.2, 0.33), turned to 90 degrees
- moved R14 18.0 mm to (-1.44, -9.46)
- moved C16 17.9 mm to (0.80, -0.44), flipped to the top
- moved R12 17.0 mm to (0.36, -9.47), flipped to the bottom
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- renumbered C35 to C31, C39 to C29, C41 to C6
Connections:
- net CAM_GPIO172: now also R7.2; no longer R13.2
- net CAM_GPIO173: now also R8.2; no longer R14.2
- net CAM_PCLK: now also R21.2; no longer R30.2
- net GND: now also C1.1, C11.2, C15.2, C17.2, C19.1, C2.1, C20.1, C21.1, C23.2, C3.1, C30.1, C33.2, C4.2, C5.1, R23.1, R24.1; no longer C1.2, C11.1, C15.1, C2.2, C20.2, C21.2, C23.1, C3.2, C33.1, C34.1, C36.1, C37.1, C40.1, C5.2, R25.1, R9.1
- net I2C_SCL: now also R4.1; no longer R16.1
- net I2C_SDA: now also R3.1; no longer R27.1
- net N$10: now also R13.1; no longer R15.1
- net N$11: now also R13.2; no longer R15.2
- net N$12: now also R14.1; no longer R5.1
- net N$14: now also R14.2; no longer R5.2
- net N$15: now also R2.2; no longer R31.2
- net N$16: now also R2.1; no longer R31.1
- net N$2: now also R9.1; no longer R4.1
- net N$21: now also C8.2; no longer C22.2
- net N$22: now also R15.1; no longer R19.1
- net N$23: now also R22.1, R23.2; no longer R8.1, R9.2
- net N$24: now also R15.2; no longer R19.2
- net N$25: now also R5.1; no longer R32.1
- net N$26: now also R5.2; no longer R32.2
- net N$3: now also R9.2; no longer R4.2
- net N$30: now also R25.1; no longer R11.1
- net N$31: now also R24.2; no longer R25.2
- net N$32: now also R7.1; no longer R13.1
- net N$33: now also R8.1; no longer R14.1
- net N$34: now also D2.A; no longer D1.A
- net N$39: now also D1.A; no longer D2.A
- net N$4: now also R10.1; no longer R17.1
- net N$40: now also R16.1; no longer R3.1
- net N$41: now also R16.2; no longer R3.2
- net N$42: now also R17.1; no longer R28.1
- net N$43: now also R17.2; no longer R28.2
- net N$44: now also R18.1; no longer R1.1
- net N$45: now also R18.2; no longer R1.2
- net N$46: now also R19.1; no longer R2.1
- net N$47: now also R19.2; no longer R2.2
- net N$48: now also R20.1; no longer R21.1
- net N$49: now also R20.2; no longer R21.2
- net N$5: now also R10.2; no longer R17.2
- net N$52: now also R6.1; no longer R12.1
- net N$6: now also R11.1; no longer R6.1
- net N$7: now also R11.2; no longer R6.2
- net N$8: now also R12.1; no longer R7.1
- net N$9: now also R12.2; no longer R7.2
- net P1P8V: now also C10.2, C11.1, C12.2, C13.2, C17.1, C28.2, C3.2, C4.1, C5.2, R1.2, R3.2, R4.2, R6.2; no longer C1.1, C14.2, C20.1, C21.1, C33.2, C34.2, C36.2, C40.2, C8.2, R10.2, R12.2, R16.2, R27.2
- net P2P8V: now also C15.1, C16.2, C19.2, C21.2, C22.2, C23.1, C24.2, C25.2, R22.2; no longer C10.2, C11.2, C12.2, C13.2, C3.1, C32.2, C5.1, C9.2, R8.2
- net P3P3V: now also C1.2, C14.2, C30.2, C32.2, C9.2; no longer C15.2, C16.2, C24.2, C28.2, C37.2
- net P5V: now also C2.2, C20.2, C33.1, R25.2; no longer C2.1, C23.2, C25.2, R11.2
- net PIXCLK: now also R21.1; no longer R30.1
- net SLA_RESET_BAR: now also R1.1; no longer R10.1

Commit message: Update SLA1500 CAM V6
Parts:
- moved R19 0.72 mm to (-7.16, -5.63)
- moved R17 0.28 mm to (-5.33, -6.06)
- moved C15 0.20 mm to (2.34, -1.66)
Routing:
- net GND: track 18.5 -> 16.9 mm, vias 8 -> 9
- net N$36: track 21.5 -> 20.1 mm
- net P5V: track 14.2 -> 15.6 mm, vias 7 -> 8
- net N$41: track 27.2 -> 28.5 mm
- net N$18: track 8.70 -> 7.89 mm
- net N$46: track 7.12 -> 6.44 mm
- net CAM_GPIO172: track 24.3 -> 23.7 mm
- net CAM_GPIO173: track 41.0 -> 41.5 mm
- net CAM_GPIO178: track 30.3 -> 29.8 mm
- net FRAME_VALID: track 48.1 -> 47.5 mm
- net P1P8V: track 41.0 -> 40.5 mm
- added copper zone on layer 1, net 0
- added copper zone on layer 16, net 0

Commit message: Update SLA1500 CAM V6
Parts:
- moved R21 3.14 mm to (-3.39, 1.98)
- moved C5 1.31 mm to (-3.44, 1.02)
- moved C7 1.29 mm to (-3.43, -0.21)
- moved R9 0.99 mm to (3.00, -3.52)
- moved U1 0.96 mm to (0.96, -0.03)
- moved C16 0.86 mm to (0.96, -1.28)
- moved C26 0.77 mm to (5.51, -1.84)
- moved C22 0.76 mm to (5.52, -0.08)
- moved C25 0.76 mm to (5.50, -0.96)
- moved C19 0.75 mm to (5.49, 1.68)
- moved C21 0.72 mm to (5.48, 0.80)
- moved R15 0.64 mm to (-0.66, -4.46)
- moved C15 0.50 mm to (2.67, -1.29)
- moved C23 0.28 mm to (2.63, 1.75)
- moved R11 0.07 mm to (1.19, -3.52)
Routing:
- net CAM_PCLK: track 22.4 -> 27.0 mm
- net CAM_GPIO178: track 29.8 -> 26.5 mm, vias 5 -> 3
- net P1P8V: track 40.5 -> 42.8 mm
- net P2P8V: track 22.7 -> 24.8 mm
- net I2C_SDA: track 22.3 -> 20.8 mm
- net N$3: track 4.93 -> 6.05 mm
- net N$22: track 2.44 -> 3.44 mm
- net N$29: track 8.18 -> 9.14 mm
- net N$44: track 2.14 -> 3.10 mm
- net N$42: track 4.84 -> 5.80 mm
- net N$40: track 2.14 -> 3.08 mm
- net N$48: track 2.17 -> 3.11 mm
- net N$46: track 6.44 -> 7.33 mm
- net I2C_SCL: track 25.9 -> 26.7 mm
- net N$2: track 2.42 -> 3.22 mm
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