File: EAGLE files/Projects/SLA_1500_CAM_V6.sch (EAGLE design)
At the start: 92 parts, among them J2 JST GH SM06B, J3 MOLEX 53261-03, J4 MOLEX 53261-04, J5 MOLEX 53261-04, J6 MOLEX 53261-04, U10 TPS73633DBVR, U11 TXS0102, U8 TXS0102, U9 TXS0102

Commit message: Update SLA1500 CAM V6
Parts:
- added C28: 100nF, Seeed-Capacitor:CERAMIC 100NF-10V-10%-X5R(0402)
- added C29: 10nf, Seeed-Capacitor:CERAMIC-10NF-50V-10%-X7R(0402)
- added R25: 0R, Seeed-Resistor:SMD-RES-0R-5%-1/16W(0402)
- added R27: 1.5K, Seeed-Resistor:SMD-RES-1.5K-5%-1/16W(0402)
- added R28: 22R, Seeed-Resistor:SMD-RES-22R-1%-1/16W(0402)
- added R29: (no value), resistor:R-EU_R0402
Changed lines of the file:
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@@
 <part name="TP3" library="testpad" library_urn="urn:adsk.eagle:library:385" deviceset="PTR1" device="TP08SQ" package3d_urn="urn:adsk.eagle:package:27960/1"/>
 <part name="U$1" library="Sightline" deviceset="HEADER_V5" device=""/>
+<part name="C28" library="Seeed-Capacitor" library_urn="urn:adsk.eagle:library:464" deviceset="CERAMIC 100NF-10V-10%-X5R(0402)" device="" package3d_urn="urn:adsk.eagle:package:32379/1" value="100nF "/>
+<part name="C29" library="Seeed-Capacitor" library_urn="urn:adsk.eagle:library:464" deviceset="CERAMIC-10NF-50V-10%-X7R(0402)" device="" package3d_urn="urn:adsk.eagle:package:32379/1" value="10nf"/>
+<part name="R25" library="Seeed-Resistor" library_urn="urn:adsk.eagle:library:474" deviceset="SMD-RES-0R-5%-1/16W(0402)" device="" package3d_urn="urn:adsk.eagle:package:32792/1" value="0R"/>
+<part name="R27" library="Seeed-Resistor" library_urn="urn:adsk.eagle:library:474" deviceset="SMD-RES-1.5K-5%-1/16W(0402)" device="" package3d_urn="urn:adsk.eagle:package:32792/1" value="1.5K"/>
+<part name="R28" library="Seeed-Resistor" library_urn="urn:adsk.eagle:library:474" deviceset="SMD-RES-22R-1%-1/16W(0402)" device="" package3d_urn="urn:adsk.eagle:package:32792/1" value="22R"/>
+<part name="R29" library="resistor" library_urn="urn:adsk.eagle:library:348" deviceset="R-EU_" device="R0402" package3d_urn="urn:adsk.eagle:package:26058/1"/>
 </parts>
 <sheets>
@@
 </instance>
 <instance part="U$1" gate="G$1" x="322.58" y="5.08" smashed="yes"/>
+<instance part="C28" gate="G$1" x="299.72" y="132.08" smashed="yes" rot="R90">
+<attribute name="NAME" x="300.99" y="133.35" size="1.27" layer="95" ratio="10"/>
+<attribute name="VALUE" x="300.99" y="129.54" size="1.27" layer="96" ratio="10"/>
+</instance>
+<instance part="C29" gate="G$1" x="299.72" y="116.84" smashed="yes" rot="R90">
+<attribute name="NAME" x="300.99" y="118.11" size="1.27" layer="95" ratio="10"/>
+<attribute name="VALUE" x="300.99" y="114.3" size="1.27" layer="96" ratio="10"/>
+</instance>
+<instance part="R25" gate="G$1" x="302.26" y="109.22" smashed="yes">
+<attribute name="NAME" x="298.45" y="110.49" size="1.27" layer="95" ratio="10"/>
+<attribute name="VALUE" x="298.45" y="106.68" size="1.27" layer="96" ratio="10"/>
+</instance>
+<instance part="R27" gate="G$1" x="297.18" y="101.6" smashed="yes">
+<attribute name="NAME" x="293.37" y="102.87" size="1.27" layer="95" ratio="10"/>
+<attribute name="VALUE" x="293.37" y="99.06" size="1.27" layer="96" ratio="10"/>
+</instance>
+<instance part="R28" gate="G$1" x="297.18" y="93.98" smashed="yes">
+<attribute name="NAME" x="293.37" y="95.25" size="1.27" layer="95" ratio="10"/>
+<attribute name="VALUE" x="293.37" y="91.44" size="1.27" layer="96" ratio="10"/>
+</instance>
+<instance part="R29" gate="G$1" x="299.72" y="86.36" smashed="yes">
+<attribute name="NAME" x="295.91" y="87.8586" size="1.778" layer="95"/>
+<attribute name="VALUE" x="295.91" y="83.058" size="1.778" layer="96"/>
+</instance>
 </instances>
 <busses>
