File: EAGLE files/Projects/SLA_1500_CAM_V6.sch (EAGLE design)
At the start: 92 parts, among them J2 JST GH SM06B, J3 MOLEX 53261-03, J4 MOLEX 53261-04, J5 MOLEX 53261-04, J6 MOLEX 53261-04, U10 TPS73633DBVR, U11 TXS0102, U8 TXS0102, U9 TXS0102

Commit message: Update SLA1500 CAM V6
Parts:
- removed C17, C19, C4, C6: 10uf, Sightline:F980G106MUA
- removed C38: 10uf, Seeed-Capacitor:TANTALUM-SMD-10UF-10V-10%(AVX-A)
- C2: device Sightline:F980G106MUA -> Sightline:F980J106MUALZT
Connections:
- net GND: no longer C17.P$2, C19.P$2, C38.-, C4.P$2, C6.P$2
- net P1P8V: no longer C19.P$1, C6.P$1
- net P2P8V: no longer C17.P$1, C2.P$1, C4.P$1
- net P5V: now also C2.P$1; no longer C38.+
Other:
- moved on the sheet: C1, C10, C11, C12, C13, C14, C18, C2, C20, C3, C32, C33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

Commit message: Update SLA1500 CAM V6
Parts:
- removed C34, C36, C37, C40: 100nF, Seeed-Capacitor:CERAMIC 100NF-10V-10%-X5R(0402)
- removed R27: 1.5K, Seeed-Resistor:SMD-RES-1.5K-5%-1/16W(0402)
- removed R28, R30, R31, R32: 22R, Seeed-Resistor:SMD-RES-22R-1%-1/16W(0402)
- added C17: 470nF, SparkFun-Capacitors:470NF-0402-16V-10%
- added C19, C30: 100nF, Seeed-Capacitor:CERAMIC 100NF-10V-10%-X5R(0402)
- added C4: 10uf, Sightline:F980G106MUA
- added R18, R20: 22R, Seeed-Resistor:SMD-RES-22R-1%-1/16W(0402)
- added R22: 60.2K, SparkFun-Resistors:62KOHM-0603-1/10W-5%
- added R23: 10k, SparkFun-Resistors:10KOHM-0603-1/10W-1%
- added R24: 0R, Seeed-Resistor:SMD-RES-0R-5%-1/16W(0402)
- C1, C3, C5: value 10uf -> 100nF; device Sightline:F980G106MUA -> Seeed-Capacitor:CERAMIC 100NF-10V-10%-X5R(0402)
- C11, C15: value 100nF -> 10uf; device Seeed-Capacitor:CERAMIC 100NF-10V-10%-X5R(0402) -> Sightline:F980G106MUA
- C2: value 10uf -> 1uf; device Sightline:F980J106MUALZT -> Seeed-Capacitor:CERAMIC-1UF-10V-10%-X5R(0402)
- C20: value 10uf -> 1uf; device Sightline:F980G106MUA -> Seeed-Capacitor:CERAMIC-1UF-10V-10%-X5R(0402)
- C21: value 470nF -> 100nF; device SparkFun-Capacitors:470NF-0402-16V-10% -> Seeed-Capacitor:CERAMIC 100NF-10V-10%-X5R(0402)
- C22: value 10nf -> 100nF; device Seeed-Capacitor:CERAMIC-10NF-50V-10%-X7R(0402) -> Seeed-Capacitor:CERAMIC 100NF-10V-10%-X5R(0402)
- C23: value 1uf -> 10uf; device Seeed-Capacitor:CERAMIC-1UF-10V-10%-X5R(0402) -> Sightline:F980G106MUA
- C25, C26: value 1uf -> 100nF; device Seeed-Capacitor:CERAMIC-1UF-10V-10%-X5R(0402) -> Seeed-Capacitor:CERAMIC 100NF-10V-10%-X5R(0402)
- C33: value 100nF -> 10uf; device Seeed-Capacitor:CERAMIC 100NF-10V-10%-X5R(0402) -> Sightline:F980J106MUALZT
- C8: value 100nF -> 10nf; device Seeed-Capacitor:CERAMIC 100NF-10V-10%-X5R(0402) -> Seeed-Capacitor:CERAMIC-10NF-50V-10%-X7R(0402)
- C9: value 100nF -> 1uf; device Seeed-Capacitor:CERAMIC 100NF-10V-10%-X5R(0402) -> Seeed-Capacitor:CERAMIC-1UF-10V-10%-X5R(0402)
- R1: value 22R -> 10k; device Seeed-Resistor:SMD-RES-22R-1%-1/16W(0402) -> SparkFun-Resistors:10KOHM-0603-1/10W-1%
- R10, R9: value 10k -> 22R; device SparkFun-Resistors:10KOHM-0603-1/10W-1% -> Seeed-Resistor:SMD-RES-22R-1%-1/16W(0402)
- R11: value 680 -> 22R; device SparkFun-Resistors:680OHM-0603-1/10W-5% -> Seeed-Resistor:SMD-RES-22R-1%-1/16W(0402)
- R12, R13, R14: value 0R -> 22R; device Seeed-Resistor:SMD-RES-0R-5%-1/16W(0402) -> Seeed-Resistor:SMD-RES-22R-1%-1/16W(0402)
- R16: value 1.5K -> 22R; device Seeed-Resistor:SMD-RES-1.5K-5%-1/16W(0402) -> Seeed-Resistor:SMD-RES-22R-1%-1/16W(0402)
- R25: value 0R -> 680; device Seeed-Resistor:SMD-RES-0R-5%-1/16W(0402) -> SparkFun-Resistors:680OHM-0603-1/10W-5%
- R3, R4: value 22R -> 1.5K; device Seeed-Resistor:SMD-RES-22R-1%-1/16W(0402) -> Seeed-Resistor:SMD-RES-1.5K-5%-1/16W(0402)
- R6, R7: value 22R -> 0R; device Seeed-Resistor:SMD-RES-22R-1%-1/16W(0402) -> Seeed-Resistor:SMD-RES-0R-5%-1/16W(0402)
- R8: value 60.2K -> 0R; device SparkFun-Resistors:62KOHM-0603-1/10W-5% -> Seeed-Resistor:SMD-RES-0R-5%-1/16W(0402)
- renumbered C35 to C31, C39 to C29, C41 to C6
Connections:
- net CAM_GPIO172: now also R7.2; no longer R13.2
- net CAM_GPIO173: now also R8.2; no longer R14.2
- net CAM_PCLK: now also R21.2; no longer R30.2
- net GND: now also C1.1, C11.P$2, C15.P$2, C17.2, C19.1, C2.1, C20.1, C21.1, C23.P$2, C3.1, C30.1, C33.P$2, C4.P$2, C5.1, R23.1, R24.1; no longer C1.P$2, C11.1, C15.1, C2.P$2, C20.P$2, C21.2, C23.1, C3.P$2, C33.1, C34.1, C36.1, C37.1, C40.1, C5.P$2, R25.1, R9.1
- net I2C_SCL: now also R4.1; no longer R16.1
- net I2C_SDA: now also R3.1; no longer R27.1
- net N$10: now also R13.1; no longer R15.1
- net N$11: now also R13.2; no longer R15.2
- net N$12: now also R14.1; no longer R5.1
- net N$14: now also R14.2; no longer R5.2
- net N$15: now also R2.2; no longer R31.2
- net N$16: now also R2.1; no longer R31.1
- net N$2: now also R9.1; no longer R4.1
- net N$21: now also C8.2; no longer C22.2
- net N$22: now also R15.1; no longer R19.1
- net N$23: now also R22.1, R23.2; no longer R8.1, R9.2
- net N$24: now also R15.2; no longer R19.2
- net N$25: now also R5.1; no longer R32.1
- net N$26: now also R5.2; no longer R32.2
- net N$3: now also R9.2; no longer R4.2
- net N$30: now also R25.1; no longer R11.1
- net N$31: now also R24.2; no longer R25.2
- net N$32: now also R7.1; no longer R13.1
- net N$33: now also R8.1; no longer R14.1
- net N$34: now also D2.A; no longer D1.A
- net N$39: now also D1.A; no longer D2.A
- net N$4: now also R10.1; no longer R17.1
- net N$40: now also R16.1; no longer R3.1
- net N$41: now also R16.2; no longer R3.2
- net N$42: now also R17.1; no longer R28.1
- net N$43: now also R17.2; no longer R28.2
- net N$44: now also R18.1; no longer R1.1
- net N$45: now also R18.2; no longer R1.2
- net N$46: now also R19.1; no longer R2.1
- net N$47: now also R19.2; no longer R2.2
- net N$48: now also R20.1; no longer R21.1
- net N$49: now also R20.2; no longer R21.2
- net N$5: now also R10.2; no longer R17.2
- net N$52: now also R6.1; no longer R12.1
- net N$6: now also R11.1; no longer R6.1
- net N$7: now also R11.2; no longer R6.2
- net N$8: now also R12.1; no longer R7.1
- net N$9: now also R12.2; no longer R7.2
- net P1P8V: now also C10.2, C11.P$1, C12.2, C13.2, C17.1, C28.2, C3.2, C4.P$1, C5.2, R1.2, R3.2, R4.2, R6.2; no longer C1.P$1, C14.2, C20.P$1, C21.1, C33.2, C34.2, C36.2, C40.2, C8.2, R10.2, R12.2, R16.2, R27.2
- net P2P8V: now also C15.P$1, C16.2, C19.2, C21.2, C22.2, C23.P$1, C24.2, C25.2, R22.2; no longer C10.2, C11.2, C12.2, C13.2, C3.P$1, C32.2, C5.P$1, C9.2, R8.2
- net P3P3V: now also C1.2, C14.2, C30.2, C32.2, C9.2; no longer C15.2, C16.2, C24.2, C28.2, C37.2
- net P5V: now also C2.2, C20.2, C33.P$1, R25.2; no longer C2.P$1, C23.2, C25.2, R11.2
- net PIXCLK: now also R21.1; no longer R30.1
- net SLA_RESET_BAR: now also R1.1; no longer R10.1
Other:
- moved on the sheet: C10, C12, C13, C14, C16, C18, C22, C24, C25, C26, C27, C28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
