File: EAGLE files/Projects/SLA_1500_CAM_V7.brd (EAGLE design)
At the start: 37.8 x 26.4 mm, 89 parts, among them J2 JST GH SM06B, J3 MOLEX 53261-03, J4 MOLEX 53261-04, J5 MOLEX 53261-04, J6 MOLEX 53261-04, U10 TPS73633DBVR, U11 TXS0102, U8 TXS0102, U9 TXS0102

Commit message: Update SLA1500CAM V7
Routing:
- net CAM_GPIO178: track 36.0 -> 36.5 mm
- net GND: vias 10 -> 22
