File: EAGLE files/Projects/SLA_1500_CAM_V8.sch (EAGLE design)
At the start: 89 parts, among them J2 JST GH SM06B, J3 MOLEX 53261-03, J4 MOLEX 53261-04, J5 MOLEX 53261-04, J6 MOLEX 53261-04, U10 TPS73633DBVR, U11 TXS0102, U8 TXS0102, U9 TXS0102

Commit message: Update Final Documentation
Changed lines of the file:
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@@
 <part name="R26" library="Seeed-Resistor" library_urn="urn:adsk.eagle:library:474" deviceset="SMD-RES-0R-5%-1/16W(0402)" device="" package3d_urn="urn:adsk.eagle:package:32792/1" value="0R"/>
 <part name="R27" library="Seeed-Resistor" library_urn="urn:adsk.eagle:library:474" deviceset="SMD-RES-0R-5%-1/16W(0402)" device="" package3d_urn="urn:adsk.eagle:package:32792/1" value="0R"/>
-<part name="U$1" library="Sightline" deviceset="HEADER_V7" device=""/>
+<part name="U$1" library="Sightline" deviceset="HEADER_V8" device=""/>
 </parts>
 <sheets>
@@
 <attribute name="VALUE" x="120.6246" y="98.8314" size="1.27" layer="96" ratio="10" rot="R270"/>
 </instance>
-<instance part="U$1" gate="G$1" x="322.58" y="5.08" smashed="yes"/>
+<instance part="U$1" gate="G$1" x="320.04" y="5.08" smashed="yes"/>
 </instances>
 <busses>
